File: pcb/vegas.kicad_pcb (KiCad board)
At the start: 2 copper layers, 304.8 x 95.2 mm, 157 parts, among them SW1 SW_Push, SW10 SW_Push, SW11 SW_Push, SW12 SW_Push, SW13 SW_Push, SW14 SW_Push, SW15 SW_Push, SW16 SW_Push, SW17 SW_Push, SW18 SW_Push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

Commit message: v0.1.0 final
Other:
- outline, holes or cut-outs redrawn
- board text added: "JLCJLCJLCJLC"
